File: _autosave-F14-DDP.kicad_pcb (KiCad board)
At the start: 2 copper layers, 21 parts, among them SW1 SW_Push, U1 ProMicro

Commit message: traces
Parts:
- added MX8: MX-NoLED, MX_Only:MXOnly-1U-NoLED, F.Cu at (188.9, 92.1)
- SW1: moved to B.Cu
- moved MX1 83.7 mm to (141.3, 49.2)
- moved D1 83.1 mm to (152.4, 50.0), turned to 90 degrees
- moved D4 76.3 mm to (152.4, 73.8), turned to 90 degrees
- moved D2 71.9 mm to (176.2, 50.0), turned to 90 degrees
- moved MX4 69.1 mm to (141.3, 73.0)
- moved SW1 68.6 mm to (243.3, 47.0), turned to 90 degrees
- moved MX3 64.4 mm to (188.9, 49.2)
- moved D3 64.4 mm to (200.0, 50.0), turned to 90 degrees
- moved MX2 62.8 mm to (165.1, 49.2)
- moved D5 54.6 mm to (176.2, 73.8), turned to 90 degrees
- moved MX5 50.9 mm to (165.1, 73.0)
- moved D6 48.8 mm to (197.6, 73.8), turned to 90 degrees
- moved D10 48.0 mm to (235.7, 80.2)
- moved MX9 43.6 mm to (212.7, 92.1)
- moved MX7 42.5 mm to (212.7, 73.0)
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Connections:
- U1 pad 13: unconnected-(U1-Pad13) -> /ROW2
- U1 pad 14: unconnected-(U1-Pad14) -> /ROW1
- U1 pad 15: unconnected-(U1-Pad15) -> /ROW0
- U1 pad 16: unconnected-(U1-Pad16) -> /COL2
- U1 pad 17: unconnected-(U1-Pad17) -> /COL3
- U1 pad 18: unconnected-(U1-Pad18) -> /COL4
- U1 pad 19: unconnected-(U1-Pad19) -> /COL1
- U1 pad 20: unconnected-(U1-Pad20) -> /COL0
Routing:
- net /COL4: track 0.00 -> 85.8 mm
- net /COL1: track 0.00 -> 44.2 mm
- net /COL0: track 0.00 -> 42.2 mm
- net /COL3: track 0.00 -> 32.7 mm
- net /COL2: track 0.00 -> 26.5 mm
- net /ROW1: track 0.00 -> 23.8 mm
- net Net-(D8-Pad2): track 0.00 -> 10.8 mm
- net Net-(D7-Pad2): track 0.00 -> 10.3 mm
- net Net-(D5-Pad2): track 0.00 -> 10.3 mm
- net Net-(D4-Pad2): track 0.00 -> 10.3 mm
- net Net-(D3-Pad2): track 0.00 -> 10.3 mm
- net Net-(D2-Pad2): track 0.00 -> 10.3 mm
- net Net-(D1-Pad2): track 0.00 -> 10.3 mm
- net Net-(D9-Pad2): track 0.00 -> 10.3 mm
- net Net-(D6-Pad2): track 0.00 -> 7.94 mm
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Other:
- board outline added: 119.1 x 65.1 mm

Commit message: Decoration pt1
Connections:
- U1 pad 10: unconnected-(U1-Pad10) -> /COL4
- U1 pad 11: unconnected-(U1-Pad11) -> /COL3
- U1 pad 12: unconnected-(U1-Pad12) -> /COL2
- U1 pad 13: /ROW2 -> unconnected-(U1-Pad13)
- U1 pad 14: /ROW1 -> unconnected-(U1-Pad14)
- U1 pad 15: /ROW0 -> unconnected-(U1-Pad15)
- U1 pad 16: /COL2 -> /ROW2
- U1 pad 17: /COL3 -> /ROW1
- U1 pad 18: /COL4 -> /ROW0
Routing:
- net GND: track 0.00 -> 181.2 mm
- net Net-(SW1-Pad1): track 0.00 -> 163.7 mm
- net /ROW2: track 0.00 -> 91.8 mm
- net /ROW0: track 0.00 -> 82.1 mm
- net /ROW1: track 23.8 -> 105.6 mm
- net /COL2: track 26.5 -> 70.3 mm
- net /COL3: track 32.7 -> 72.0 mm
- net /COL4: track 85.8 -> 82.7 mm
- added copper zone on F.Cu, net GND
