File: F14-DDP.kicad_pcb (KiCad board)
At the start: 2 copper layers, 21 parts, among them SW1 SW_Push, U1 ProMicro

Commit message: Done!
Parts:
- added G***: LOGO, F14:f14, F.Cu at (219.9, 51.6)
- added MX8: MX-NoLED, MX_Only:MXOnly-1U-NoLED, F.Cu at (188.9, 92.1)
- SW1: moved to B.Cu
- moved MX1 83.7 mm to (141.3, 49.2)
- moved D1 83.1 mm to (152.4, 50.0), turned to 90 degrees
- moved D4 76.3 mm to (152.4, 73.8), turned to 90 degrees
- moved D2 71.9 mm to (176.2, 50.0), turned to 90 degrees
- moved MX4 69.1 mm to (141.3, 73.0)
- moved SW1 68.6 mm to (243.3, 47.0), turned to 90 degrees
- moved MX3 64.4 mm to (188.9, 49.2)
- moved D3 64.4 mm to (200.0, 50.0), turned to 90 degrees
- moved MX2 62.8 mm to (165.1, 49.2)
- moved D5 54.6 mm to (176.2, 73.8), turned to 90 degrees
- moved MX5 50.9 mm to (165.1, 73.0)
- moved D6 48.8 mm to (197.6, 73.8), turned to 90 degrees
- moved D10 48.0 mm to (235.7, 80.2)
- moved MX9 43.6 mm to (212.7, 92.1)
- moved MX7 42.5 mm to (212.7, 73.0)
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Connections:
- U1 pad 10: unconnected-(U1-Pad10) -> /COL4
- U1 pad 11: unconnected-(U1-Pad11) -> /COL3
- U1 pad 12: unconnected-(U1-Pad12) -> /COL2
- U1 pad 16: unconnected-(U1-Pad16) -> /ROW2
- U1 pad 17: unconnected-(U1-Pad17) -> /ROW1
- U1 pad 18: unconnected-(U1-Pad18) -> /ROW0
- U1 pad 19: unconnected-(U1-Pad19) -> /COL1
- U1 pad 20: unconnected-(U1-Pad20) -> /COL0
Routing:
- net GND: track 0.00 -> 181.2 mm
- net Net-(SW1-Pad1): track 0.00 -> 163.7 mm
- net /ROW1: track 0.00 -> 105.6 mm
- net /ROW2: track 0.00 -> 91.8 mm
- net /COL4: track 0.00 -> 82.7 mm
- net /ROW0: track 0.00 -> 82.1 mm
- net /COL3: track 0.00 -> 72.0 mm
- net /COL2: track 0.00 -> 70.3 mm
- net /COL1: track 0.00 -> 44.2 mm
- net /COL0: track 0.00 -> 42.2 mm
- net Net-(D8-Pad2): track 0.00 -> 10.8 mm
- net Net-(D7-Pad2): track 0.00 -> 10.3 mm
- net Net-(D5-Pad2): track 0.00 -> 10.3 mm
- net Net-(D4-Pad2): track 0.00 -> 10.3 mm
- net Net-(D3-Pad2): track 0.00 -> 10.3 mm
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- added copper zone on F.Cu, net GND
Other:
- board outline added: 119.1 x 65.1 mm
- board text added: "F-14 DDP by NibbledPots"

Commit message: more beautification
Parts:
- moved G*** 1.77 mm to (218.3, 52.4)
Connections:
- U1 pad 14: unconnected-(U1-Pad14) -> /COL1
- U1 pad 19: /COL1 -> unconnected-(U1-Pad19)
Routing:
- net /COL1: track 44.2 -> 38.6 mm
- net /COL3: track 72.0 -> 77.6 mm
- net /COL2: track 70.3 -> 74.1 mm
- net /COL4: track 82.7 -> 85.5 mm
- net /ROW2: track 91.8 -> 94.0 mm
- net unconnected-(U1-Pad19): track 0.00 -> 0.81 mm
Changed lines of the file:
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@@
   (net 29 "unconnected-(U1-Pad24)")
   (net 30 "unconnected-(U1-Pad13)")
-  (net 31 "unconnected-(U1-Pad14)")
+  (net 31 "unconnected-(U1-Pad19)")
   (net 32 "unconnected-(U1-Pad15)")
   (footprint "Diode_SMD:D_SOD-123" (layer "F.Cu")
@@
       (effects (font (size 1 1) (thickness 0.15)))
     )
+    (fp_line (start -7 7) (end -5 7) (layer "Dwgs.User") (width 0.15))
+    (fp_line (start -7 5) (end -7 7) (layer "Dwgs.User") (width 0.15))
+    (fp_line (start 9.525 -9.525) (end 9.525 9.525) (layer "Dwgs.User") (width 0.15))
+    (fp_line (start -9.525 9.525) (end -9.525 -9.525) (layer "Dwgs.User") (width 0.15))
+    (fp_line (start -7 -7) (end -7 -5) (layer "Dwgs.User") (width 0.15))
+    (fp_line (start 5 -7) (end 7 -7) (layer "Dwgs.User") (width 0.15))
     (fp_line (start 7 7) (end 7 5) (layer "Dwgs.User") (width 0.15))
+    (fp_line (start -9.525 -9.525) (end 9.525 -9.525) (layer "Dwgs.User") (width 0.15))
+    (fp_line (start 7 -7) (end 7 -5) (layer "Dwgs.User") (width 0.15))
     (fp_line (start -5 -7) (end -7 -7) (layer "Dwgs.User") (width 0.15))
-    (fp_line (start 9.525 -9.525) (end 9.525 9.525) (layer "Dwgs.User") (width 0.15))
-    (fp_line (start -7 -7) (end -7 -5) (layer "Dwgs.User") (width 0.15))
-    (fp_line (start -7 7) (end -5 7) (layer "Dwgs.User") (width 0.15))
-    (fp_line (start -9.525 -9.525) (end 9.525 -9.525) (layer "Dwgs.User") (width 0.15))
-    (fp_line (start -7 5) (end -7 7) (layer "Dwgs.User") (width 0.15))
+    (fp_line (start 5 7) (end 7 7) (layer "Dwgs.User") (width 0.15))
     (fp_line (start 9.525 9.525) (end -9.525 9.525) (layer "Dwgs.User") (width 0.15))
-    (fp_line (start 7 -7) (end 7 -5) (layer "Dwgs.User") (width 0.15))
-    (fp_line (start 5 -7) (end 7 -7) (layer "Dwgs.User") (width 0.15))
-    (fp_line (start -9.525 9.525) (end -9.525 -9.525) (layer "Dwgs.User") (width 0.15))
-    (fp_line (start 5 7) (end 7 7) (layer "Dwgs.User") (width 0.15))
     (pad "" np_thru_hole circle locked (at 5.08 0 48.0996) (size 1.75 1.75) (drill 1.75) (layers *.Cu *.Mask))
+    (pad "" np_thru_hole circle locked (at -5.08 0 48.0996) (size 1.75 1.75) (drill 1.75) (layers *.Cu *.Mask))
     (pad "" np_thru_hole circle locked (at 0 0) (size 3.9878 3.9878) (drill 3.9878) (layers *.Cu *.Mask))
-    (pad "" np_thru_hole circle locked (at -5.08 0 48.0996) (size 1.75 1.75) (drill 1.75) (layers *.Cu *.Mask))
     (pad "1" thru_hole circle locked (at -3.81 -2.54) (size 2.25 2.25) (drill 1.47) (layers *.Cu "B.Mask")
       (net 16 "/COL2") (pinfunction "COL") (pintype "passive"))
@@
       (net 30 "unconnected-(U1-Pad13)") (pinfunction "10/PB6") (pintype "input"))
     (pad "14" thru_hole circle locked (at 11.43 -7.62) (size 1.7526 1.7526) (drill 1.0922) (layers *.Cu *.SilkS *.Mask)
-      (net 31 "unconnected-(U1-Pad14)") (pinfunction "16/PB2") (pintype "input"))
+      (net 15 "/COL1") (pinfunction "16/PB2") (pintype "input"))
     (pad "15" thru_hole circle locked (at 8.89 -7.62) (size 1.7526 1.7526) (drill 1.0922) (layers *.Cu *.SilkS *.Mask)
       (net 32 "unconnected-(U1-Pad15)") (pinfunction "14/PB3") (pintype "input"))
@@
       (net 1 "/ROW0") (pinfunction "A1/PF6") (pintype "input"))
     (pad "19" thru_hole circle locked (at -1.27 -7.62) (size 1.7526 1.7526) (drill 1.0922) (layers *.Cu *.SilkS *.Mask)
-      (net 15 "/COL1") (pinfunction "A2/PF5") (pintype "input"))
+      (net 31 "unconnected-(U1-Pad19)") (pinfunction "A2/PF5") (pintype "input"))
     (pad "20" thru_hole circle locked (at -3.81 -7.62) (size 1.7526 1.7526) (drill 1.0922) (layers *.Cu *.SilkS *.Mask)
       (net 14 "/COL0") (pinfunction "A3/PF4") (pintype "input"))
@@
   )
   (footprint "F14:f14" (layer "F.Cu")
-    (at 219.86875 51.59375)
+    (at 218.28125 52.3875)
     (attr board_only exclude_from_pos_files exclude_from_bom)
     (fp_text reference "G***" (at 0 0) (layer "F.SilkS") hide
@@
   (gr_line (start 246.0625 103.1875) (end 130.175 103.1875) (layer "Edge.Cuts") (width 0.1))
   (gr_arc (start 247.65 101.6) (mid 247.185032 102.722532) (end 246.0625 103.1875) (layer "Edge.Cuts") (width 0.1))
-  (gr_text "F-14 DDP\nby NibbledPots" (at 218.28125 60.325) (layer "F.SilkS")
+  (gr_text "F-14 DDP\nby NibbledPots" (at 218.28125 58.7375) (layer "F.Mask")
     (effects (font (size 2.5 2.5) (thickness 0.5)) (justify left))
   )
@@
   (segment (start 223.8375 94.51875) (end 200.025 94.51875) (width 0.254) (layer "F.Cu") (net 10))
   (segment (start 227.0125 92.86875) (end 225.3625 94.51875) (width 0.254) (layer "F.Cu") (net 10))
-  (segment (start 165.008439 84.045939) (end 157.571561 84.045939) (width 0.254) (layer "F.Cu") (net 10))
-  (segment (start 157.571561 84.045939) (end 156.36875 85.24875) (width 0.254) (layer "F.Cu") (net 10))
+  (segment (start 156.36875 84.1375) (end 156.36875 85.24875) (width 0.254) (layer "F.Cu") (net 10))
+  (segment (start 166.6875 84.1375) (end 165.89375 83.34375) (width 0.254) (layer "F.Cu") (net 10))
+  (segment (start 166.6875 85.725) (end 166.6875 84.1375) (width 0.254) (layer "F.Cu") (net 10))
   (segment (start 234.09375 80.16875) (end 234.09375 82.665522) (width 0.254) (layer "F.Cu") (net 10))
+  (segment (start 175.48125 94.51875) (end 166.6875 85.725) (width 0.254) (layer "F.Cu") (net 10))
   (segment (start 227.0125 89.746772) (end 227.0125 92.86875) (width 0.254) (layer "F.Cu") (net 10))
-  (segment (start 175.48125 94.51875) (end 165.008439 84.045939) (width 0.254) (layer "F.Cu") (net 10))
   (segment (start 234.09375 82.665522) (end 227.0125 89.746772) (width 0.254) (layer "F.Cu") (net 10))
   (segment (start 225.3625 94.51875) (end 223.8375 94.51875) (width 0.254) (layer "F.Cu") (net 10))
+  (segment (start 157.1625 83.34375) (end 156.36875 84.1375) (width 0.254) (layer "F.Cu") (net 10))
+  (segment (start 165.89375 83.34375) (end 157.1625 83.34375) (width 0.254) (layer "F.Cu") (net 10))
   (segment (start 200.025 94.51875) (end 175.48125 94.51875) (width 0.254) (layer "F.Cu") (net 10))
   (segment (start 195.80125 86.995) (end 200.025 91.21875) (width 0.254) (layer "F.Cu") (net 11))
@@
   (segment (start 137.4775 46.6725) (end 137.4775 70.485) (width 0.25) (layer "B.Cu") (net 14))
   (segment (start 161.29 46.6725) (end 161.29 70.485) (width 0.25) (layer "B.Cu") (net 15))
-  (segment (start 149.563341 85.24875) (end 148.74875 85.24875) (width 0.25) (layer "B.Cu") (net 15))
-  (segment (start 161.29 73.522091) (end 149.563341 85.24875) (width 0.25) (layer "B.Cu") (net 15))
-  (segment (start 161.29 70.485) (end 161.29 73.522091) (width 0.25) (layer "B.Cu") (net 15))
+  (segment (start 161.29 85.09) (end 161.44875 85.24875) (width 0.25) (layer "B.Cu") (net 15))
+  (segment (start 161.29 70.485) (end 161.29 85.09) (width 0.25) (layer "B.Cu") (net 15))
   (segment (start 185.1025 46.6725) (end 185.1025 70.485) (width 0.25) (layer "B.Cu") (net 16))
-  (segment (start 185.1025 89.535) (end 185.1025 92.572091) (width 0.25) (layer "B.Cu") (net 16))
   (segment (start 185.1025 70.485) (end 185.1025 89.535) (width 0.25) (layer "B.Cu") (net 16))
-  (segment (start 185.1025 92.572091) (end 177.185841 100.48875) (width 0.25) (layer "B.Cu") (net 16))
-  (segment (start 177.185841 100.48875) (end 163.98875 100.48875) (width 0.25) (layer "B.Cu") (net 16))
+  (segment (start 163.98875 100.48875) (end 183.67375 100.48875) (width 0.25) (layer "B.Cu") (net 16))
+  (segment (start 185.1025 99.06) (end 185.1025 89.535) (width 0.25) (layer "B.Cu") (net 16))
+  (segment (start 183.67375 100.48875) (end 185.1025 99.06) (width 0.25) (layer "B.Cu") (net 16))
+  (segment (start 208.915 89.535) (end 208.915 99.06) (width 0.25) (layer "B.Cu") (net 17))
+  (segment (start 206.285439 101.689561) (end 162.649561 101.689561) (width 0.25) (layer "B.Cu") (net 17))
   (segment (start 162.649561 101.689561) (end 161.44875 100.48875) (width 0.25) (layer "B.Cu") (net 17))
-  (segment (start 208.915 89.535) (end 207.32401 89.535) (width 0.25) (layer "B.Cu") (net 17))
-  (segment (start 195.169449 101.689561) (end 162.649561 101.689561) (width 0.25) (layer "B.Cu") (net 17))
-  (segment (start 207.32401 89.535) (end 195.169449 101.689561) (width 0.25) (layer "B.Cu") (net 17))
   (segment (start 208.915 70.485) (end 208.915 89.535) (width 0.25) (layer "B.Cu") (net 17))
-  (segment (start 224.63125 102.39375) (end 160.81375 102.39375) (width 0.254) (layer "B.Cu") (net 18))
-  (segment (start 232.7275 94.2975) (end 224.63125 102.39375) (width 0.254) (layer "B.Cu") (net 18))
-  (segment (start 232.7275 89.535) (end 232.7275 94.2975) (width 0.254) (layer "B.Cu") (net 18))
+  (segment (start 208.915 99.06) (end 206.285439 101.689561) (width 0.25) (layer "B.Cu") (net 17))
+  (segment (start 229.39375 102.39375) (end 232.7275 99.06) (width 0.254) (layer "B.Cu") (net 18))
+  (segment (start 229.39375 102.39375) (end 160.81375 102.39375) (width 0.254) (layer "B.Cu") (net 18))
+  (segment (start 232.7275 89.535) (end 232.7275 99.06) (width 0.254) (layer "B.Cu") (net 18))
   (segment (start 160.81375 102.39375) (end 158.90875 100.48875) (width 0.254) (layer "B.Cu") (net 18))
   (segment (start 141.12875 100.48875) (end 143.66875 100.48875) (width 0.381) (layer "F.Cu") (net 19))
@@
   (segment (start 243.2625 46.975) (end 238.968489 42.680989) (width 0.254) (layer "F.Cu") (net 20))
   (segment (start 130.96875 42.06875) (end 130.96875 75.08875) (width 0.254) (layer "F.Cu") (net 20))
+  (segment (start 149.563341 85.24875) (end 148.74875 85.24875) (width 0.25) (layer "B.Cu") (net 31))
   (zone (net 19) (net_name "GND") (layer "F.Cu") (hatch edge 0.508)
     (connect_pads (clearance 0.508))
