File: F14-DDP.kicad_pcb (KiCad board)
At the start: 2 copper layers, 119.1 x 65.1 mm, 23 parts, among them SW1 SW_Push, U1 ProMicro

Commit message: more deco
Parts:
- moved SW1 13.5 mm to (229.8, 46.2)
- moved G*** 10.3 mm to (208.8, 48.4)
Routing:
- net Net-(SW1-Pad1): track 165.6 -> 151.5 mm
- net GND: track 189.4 -> 175.6 mm
- net /ROW1: track 73.3 -> 74.7 mm
Other:
- board size 119.1 x 65.1 mm -> 106.4 x 65.1 mm
Changed lines of the file:
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@@
   )
   (footprint "F14:f14" (layer "F.Cu")
-    (at 218.28125 52.3875)
+    (at 208.75625 48.41875)
     (attr board_only exclude_from_pos_files exclude_from_bom)
     (fp_text reference "G***" (at 0 0) (layer "F.SilkS") hide
@@
   )
   (footprint "Keebio-Parts:SW_Tactile_SPST_Angled_MJTP1117-no-mount" (layer "B.Cu")
-    (at 243.2625 46.975 90)
+    (at 229.76875 46.18125 90)
     (descr "tactile switch SPST right angle, PTS645VL39-2 LFS")
     (tags "tactile switch SPST angled PTS645VL39-2 LFS C&K Button")
@@
   (gr_line (start 128.5875 101.6) (end 128.5875 39.6875) (layer "Edge.Cuts") (width 0.1))
   (gr_arc (start 128.5875 39.6875) (mid 129.052468 38.564968) (end 130.175 38.1) (layer "Edge.Cuts") (width 0.1))
-  (gr_line (start 247.65 39.6875) (end 247.65 101.6) (layer "Edge.Cuts") (width 0.1))
+  (gr_line (start 234.95 39.6875) (end 234.95 101.6) (layer "Edge.Cuts") (width 0.1))
   (gr_arc (start 130.175 103.1875) (mid 129.052468 102.722532) (end 128.5875 101.6) (layer "Edge.Cuts") (width 0.1))
-  (gr_arc (start 246.0625 38.1) (mid 247.185032 38.564968) (end 247.65 39.6875) (layer "Edge.Cuts") (width 0.1))
-  (gr_line (start 130.175 38.1) (end 246.0625 38.1) (layer "Edge.Cuts") (width 0.1))
-  (gr_line (start 246.0625 103.1875) (end 130.175 103.1875) (layer "Edge.Cuts") (width 0.1))
-  (gr_arc (start 247.65 101.6) (mid 247.185032 102.722532) (end 246.0625 103.1875) (layer "Edge.Cuts") (width 0.1))
-  (gr_text "F-14 DDP\nby NibbledPots" (at 218.28125 65.0875) (layer "F.Mask")
-    (effects (font (size 2.5 2.5) (thickness 0.5)) (justify left))
+  (gr_arc (start 233.3625 38.1) (mid 234.485032 38.564968) (end 234.95 39.6875) (layer "Edge.Cuts") (width 0.1))
+  (gr_line (start 130.175 38.1) (end 233.3625 38.1) (layer "Edge.Cuts") (width 0.1))
+  (gr_line (start 233.3625 103.1875) (end 130.175 103.1875) (layer "Edge.Cuts") (width 0.1))
+  (gr_arc (start 234.95 101.6) (mid 234.485032 102.722532) (end 233.3625 103.1875) (layer "Edge.Cuts") (width 0.1))
+  (gr_text "F-14 DDP\nby NibbledPots" (at 206.375 57.94375) (layer "F.Mask")
+    (effects (font (size 2.4 2.4) (thickness 0.5)) (justify left))
   )
   (segment (start 149.092239 82.258489) (end 151.28875 84.455) (width 0.254) (layer "F.Cu") (net 1))
@@
   (segment (start 192.88125 46.0375) (end 192.88125 48.35625) (width 0.254) (layer "F.Cu") (net 4))
   (segment (start 190.97625 44.1325) (end 192.88125 46.0375) (width 0.254) (layer "F.Cu") (net 4))
-  (segment (start 150.01875 76.99375) (end 153.82875 80.80375) (width 0.254) (layer "F.Cu") (net 5))
-  (segment (start 150.01875 75.46875) (end 150.01875 76.99375) (width 0.254) (layer "F.Cu") (net 5))
+  (segment (start 150.8125 82.55) (end 153.19375 82.55) (width 0.254) (layer "F.Cu") (net 5))
+  (segment (start 150.01875 75.46875) (end 150.01875 81.75625) (width 0.254) (layer "F.Cu") (net 5))
+  (segment (start 153.19375 82.55) (end 153.82875 83.185) (width 0.254) (layer "F.Cu") (net 5))
+  (segment (start 153.82875 83.185) (end 153.82875 84.455) (width 0.254) (layer "F.Cu") (net 5))
+  (segment (start 150.01875 81.75625) (end 150.8125 82.55) (width 0.254) (layer "F.Cu") (net 5))
   (segment (start 212.725 75.46875) (end 150.01875 75.46875) (width 0.254) (layer "F.Cu") (net 5))
-  (segment (start 153.82875 80.80375) (end 153.82875 84.455) (width 0.254) (layer "F.Cu") (net 5))
   (segment (start 148.11375 67.945) (end 150.01875 69.85) (width 0.254) (layer "F.Cu") (net 6))
   (segment (start 150.01875 69.85) (end 150.01875 72.16875) (width 0.254) (layer "F.Cu") (net 6))
@@
   (segment (start 143.66875 99.695) (end 143.66875 94.77375) (width 0.381) (layer "F.Cu") (net 19))
   (segment (start 143.66875 94.77375) (end 141.12875 92.23375) (width 0.381) (layer "F.Cu") (net 19))
+  (segment (start 229.76875 41.18125) (end 226.91875 41.18125) (width 0.381) (layer "B.Cu") (net 19))
   (segment (start 130.175 80.16875) (end 130.96875 80.9625) (width 0.381) (layer "B.Cu") (net 19))
   (segment (start 131.7625 39.6875) (end 130.175 41.275) (width 0.381) (layer "B.Cu") (net 19))
   (segment (start 136.525 80.9625) (end 138.58875 83.02625) (width 0.381) (layer "B.Cu") (net 19))
+  (segment (start 226.91875 41.18125) (end 225.425 39.6875) (width 0.381) (layer "B.Cu") (net 19))
   (segment (start 130.175 41.275) (end 130.175 80.16875) (width 0.381) (layer "B.Cu") (net 19))
   (segment (start 138.58875 83.02625) (end 138.58875 84.455) (width 0.381) (layer "B.Cu") (net 19))
-  (segment (start 243.2625 41.975) (end 240.4125 41.975) (width 0.381) (layer "B.Cu") (net 19))
-  (segment (start 238.125 39.6875) (end 131.7625 39.6875) (width 0.381) (layer "B.Cu") (net 19))
-  (segment (start 240.4125 41.975) (end 238.125 39.6875) (width 0.381) (layer "B.Cu") (net 19))
+  (segment (start 225.425 39.6875) (end 131.7625 39.6875) (width 0.381) (layer "B.Cu") (net 19))
   (segment (start 130.96875 80.9625) (end 136.525 80.9625) (width 0.381) (layer "B.Cu") (net 19))
+  (segment (start 229.76875 46.18125) (end 227.95 46.18125) (width 0.254) (layer "B.Cu") (net 20))
   (segment (start 131.7625 41.275) (end 131.7625 79.375) (width 0.254) (layer "B.Cu") (net 20))
-  (segment (start 243.2625 46.975) (end 238.125 41.8375) (width 0.254) (layer "B.Cu") (net 20))
   (segment (start 141.12875 82.39125) (end 141.12875 84.455) (width 0.254) (layer "B.Cu") (net 20))
-  (segment (start 238.125 41.8375) (end 238.125 41.275) (width 0.254) (layer "B.Cu") (net 20))
+  (segment (start 227.95 46.18125) (end 222.25 40.48125) (width 0.254) (layer "B.Cu") (net 20))
+  (segment (start 222.25 40.48125) (end 132.55625 40.48125) (width 0.254) (layer "B.Cu") (net 20))
   (segment (start 132.55625 40.48125) (end 131.7625 41.275) (width 0.254) (layer "B.Cu") (net 20))
   (segment (start 132.55625 80.16875) (end 138.90625 80.16875) (width 0.254) (layer "B.Cu") (net 20))
   (segment (start 138.90625 80.16875) (end 141.12875 82.39125) (width 0.254) (layer "B.Cu") (net 20))
-  (segment (start 237.33125 40.48125) (end 132.55625 40.48125) (width 0.254) (layer "B.Cu") (net 20))
-  (segment (start 238.125 41.275) (end 237.33125 40.48125) (width 0.254) (layer "B.Cu") (net 20))
   (segment (start 131.7625 79.375) (end 132.55625 80.16875) (width 0.254) (layer "B.Cu") (net 20))
   (zone (net 19) (net_name "GND") (layer "F.Cu") (hatch edge 0.508)
@@
     (polygon
       (pts
-        (xy 247.65 103.1875)
+        (xy 234.95 103.1875)
         (xy 128.5875 103.1875)
         (xy 128.5875 38.1)
-        (xy 247.65 38.1)
+        (xy 234.95 38.1)
       )
     )

Commit message: back filling
Parts:
- added G***: LOGO, F14:F14firing, B.Cu at (212.5, 51.8)
Routing:
- added copper zone on B.Cu, net GND
