File: F14-DDP.kicad_pcb (KiCad board)
At the start: 2 copper layers, 106.4 x 65.1 mm, 24 parts, among them SW1 SW_Push, U1 ProMicro

Commit message: cleaned up traces
Parts:
- moved G*** 3.97 mm to (208.8, 52.4)
- moved G*** 3.42 mm to (215.9, 51.8)
Routing:
- net /ROW2: track 82.2 -> 84.6 mm
- net Net-(SW1-Pad1): track 151.5 -> 153.5 mm
- net GND: track 175.6 -> 174.2 mm
- net /COL2: track 68.1 -> 69.0 mm
- net Net-(D10-Pad2): track 4.35 -> 5.24 mm
Other:
- board size 106.4 x 65.1 mm -> 106.4 x 65.9 mm

Commit message: edited fillings
Changed lines of the file:
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@@
   (segment (start 227.0125 45.24375) (end 227.0125 41.275) (width 0.254) (layer "F.Cu") (net 20))
   (segment (start 226.21875 40.48125) (end 132.55625 40.48125) (width 0.254) (layer "F.Cu") (net 20))
-  (zone (net 19) (net_name "GND") (layer "F.Cu") (hatch edge 0.508)
+  (zone (net 19) (net_name "GND") (layers F&B.Cu) (hatch edge 0.508)
     (connect_pads (clearance 0.508))
     (min_thickness 0.254) (filled_areas_thickness no)
@@
         (xy 234.95 103.98125)
         (xy 128.5875 103.98125)
-        (xy 128.5875 38.89375)
-        (xy 234.95 38.89375)
+        (xy 128.5875 38.1)
+        (xy 234.95 38.1)
       )
     )
-  )
-  (zone (net 19) (net_name "GND") (layer "B.Cu") (hatch edge 0.508)
-    (connect_pads (clearance 0.508))
-    (min_thickness 0.254) (filled_areas_thickness no)
-    (fill yes (thermal_gap 0.508) (thermal_bridge_width 0.508))
-    (polygon
-      (pts
-        (xy 234.95 103.98125)
-        (xy 128.5875 103.98125)
-        (xy 128.5875 38.89375)
-        (xy 234.95 38.89375)
-      )
-    )

Commit message: v2 changes
Parts:
- moved U1 82.9 mm to (224.6, 56.0), turned to -90 degrees
- moved G*** 74.6 mm to (146.1, 92.9)
- moved G*** 71.4 mm to (156.4, 91.3)
- moved SW1 18.5 mm to (212.1, 40.9), turned to 180 degrees
Connections:
- U1 pad 10: /COL4 -> /ROW1
- U1 pad 11: /COL3 -> unconnected-(U1-Pad11)
- U1 pad 12: /COL2 -> /COL4
- U1 pad 13: unconnected-(U1-Pad13) -> /ROW2
- U1 pad 14: /COL1 -> unconnected-(U1-Pad14)
- U1 pad 16: /ROW2 -> unconnected-(U1-Pad16)
- U1 pad 17: /ROW1 -> unconnected-(U1-Pad17)
- U1 pad 18: /ROW0 -> unconnected-(U1-Pad18)
- U1 pad 20: /COL0 -> unconnected-(U1-Pad20)
- U1 pad 5: unconnected-(U1-Pad5) -> /COL0
- U1 pad 6: unconnected-(U1-Pad6) -> /COL1
- U1 pad 7: unconnected-(U1-Pad7) -> /COL2
- U1 pad 8: unconnected-(U1-Pad8) -> /COL3
- U1 pad 9: unconnected-(U1-Pad9) -> /ROW0
Routing:
- net GND: track 174.2 -> 12.5 mm
- net Net-(SW1-Pad1): track 153.5 -> 23.5 mm
- net /COL0: track 42.0 -> 112.1 mm
- net /COL4: track 74.4 -> 20.9 mm
- net /COL1: track 39.5 -> 92.6 mm
- net /COL3: track 70.5 -> 40.3 mm
- net /ROW2: track 84.6 -> 55.3 mm
- net /COL2: track 69.0 -> 89.0 mm
- net /ROW0: track 77.7 -> 71.4 mm
- net Net-(D10-Pad2): track 5.24 -> 4.35 mm
