File: F14-DDP.kicad_sch (KiCad schematic)
At the start: 22 parts

Commit message: more beautification
Connections:
- net COL0: now also U1.20 (A3/PF4)
- net COL1: now also U1.19 (A2/PF5)
- net COL2: now also U1.12 (9/PB5)
- net COL3: now also U1.11 (8/PB4)
- net COL4: now also U1.10 (7/PE6)
- net ROW0: now also U1.18 (A1/PF6)
- net ROW1: now also U1.17 (A0/PF7)
- net ROW2: now also U1.16 (15/PB1)
Changed lines of the file:
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@@
     (effects (font (size 1.27 1.27)) (justify left))
+  )
+  (hierarchical_label "COL4" (shape input) (at 88.9 81.28 180)
+    (effects (font (size 1.27 1.27)) (justify right))
+  )
+  (hierarchical_label "COL0" (shape input) (at 124.46 68.58 0)
+    (effects (font (size 1.27 1.27)) (justify left))
+  )
+  (hierarchical_label "COL1" (shape input) (at 124.46 71.12 0)
+    (effects (font (size 1.27 1.27)) (justify left))
+  )
+  (hierarchical_label "ROW0" (shape input) (at 124.46 73.66 0)
+    (effects (font (size 1.27 1.27)) (justify left))
+  )
+  (hierarchical_label "COL2" (shape input) (at 88.9 86.36 180)
+    (effects (font (size 1.27 1.27)) (justify right))
   )
   (hierarchical_label "ROW0" (shape input) (at 160.02 54.61 180)
     (effects (font (size 1.27 1.27)) (justify right))
+  )
+  (hierarchical_label "ROW2" (shape input) (at 124.46 78.74 0)
+    (effects (font (size 1.27 1.27)) (justify left))
   )
   (hierarchical_label "COL1" (shape input) (at 196.85 30.48 90)
@@
     (effects (font (size 1.27 1.27)) (justify left))
   )
+  (hierarchical_label "COL3" (shape input) (at 88.9 83.82 180)
+    (effects (font (size 1.27 1.27)) (justify right))
+  )
+  (hierarchical_label "ROW1" (shape input) (at 124.46 76.2 0)
+    (effects (font (size 1.27 1.27)) (justify left))
+  )

Commit message: redid spacing and traces
Connections:
- net COL1: now also U1.14 (16/PB2); no longer U1.19 (A2/PF5)
Changed lines of the file:
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@@
     (effects (font (size 1.27 1.27)) (justify right))
+  )
+  (hierarchical_label "COL1" (shape input) (at 124.46 83.82 0)
+    (effects (font (size 1.27 1.27)) (justify left))
   )
   (hierarchical_label "COL0" (shape input) (at 124.46 68.58 0)
     (effects (font (size 1.27 1.27)) (justify left))
   )
-  (hierarchical_label "COL1" (shape input) (at 124.46 71.12 0)
-    (effects (font (size 1.27 1.27)) (justify left))
-  )

Commit message: v2 changes
Parts:
- D1, D10, D2, D3, D5, D6, D7, D8, D9: footprint (none) -> Diode_SMD:D_SOD-123
- D4: value (none) -> D_Small; footprint (none) -> Diode_SMD:D_SOD-123
- MX1, MX10, MX2, MX3, MX4, MX5, MX6, MX7, MX9: footprint (none) -> MX_Only:MXOnly-1U-NoLED
- SW1: value (none) -> SW_Push; footprint (none) -> Keebio-Parts:SW_Tactile_SPST_Angled_MJTP1117-no-mount
- U1: value (none) -> ProMicro; footprint (none) -> Keebio-Parts:ArduinoProMicro
Connections:
- net COL0: now also U1.5 (2/PD1); no longer U1.20 (A3/PF4)
- net COL1: now also U1.6 (3/PD0); no longer U1.14 (16/PB2)
- net COL2: now also U1.7 (4/PD4); no longer U1.12 (9/PB5)
- net COL3: now also U1.8 (5/PC6); no longer U1.11 (8/PB4)
- net COL4: now also U1.12 (9/PB5); no longer U1.10 (7/PE6)
- net ROW0: now also U1.9 (6/PD7); no longer U1.18 (A1/PF6)
- net ROW1: now also U1.10 (7/PE6); no longer U1.17 (A0/PF7)
- net ROW2: now also U1.13 (10/PB6); no longer U1.16 (15/PB1)
Changed lines of the file:
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@@
     (effects (font (size 1.27 1.27)) (justify left))
   )
-  (hierarchical_label "COL4" (shape input) (at 88.9 81.28 180)
-    (effects (font (size 1.27 1.27)) (justify right))
-  )
-  (hierarchical_label "COL1" (shape input) (at 124.46 83.82 0)
-    (effects (font (size 1.27 1.27)) (justify left))
-  )
-  (hierarchical_label "COL0" (shape input) (at 124.46 68.58 0)
-    (effects (font (size 1.27 1.27)) (justify left))
-  )
-  (hierarchical_label "ROW0" (shape input) (at 124.46 73.66 0)
-    (effects (font (size 1.27 1.27)) (justify left))
-  )
-  (hierarchical_label "COL2" (shape input) (at 88.9 86.36 180)
+  (hierarchical_label "COL4" (shape input) (at 88.9 86.36 180)
+    (effects (font (size 1.27 1.27)) (justify right))
+  )
+  (hierarchical_label "COL1" (shape input) (at 88.9 71.12 180)
+    (effects (font (size 1.27 1.27)) (justify right))
+  )
+  (hierarchical_label "COL0" (shape input) (at 88.9 68.58 180)
+    (effects (font (size 1.27 1.27)) (justify right))
+  )
+  (hierarchical_label "ROW0" (shape input) (at 88.9 78.74 180)
+    (effects (font (size 1.27 1.27)) (justify right))
+  )
+  (hierarchical_label "COL2" (shape input) (at 88.9 73.66 180)
     (effects (font (size 1.27 1.27)) (justify right))
   )
@@
     (effects (font (size 1.27 1.27)) (justify right))
   )
-  (hierarchical_label "ROW2" (shape input) (at 124.46 78.74 0)
+  (hierarchical_label "ROW2" (shape input) (at 124.46 86.36 0)
     (effects (font (size 1.27 1.27)) (justify left))
   )
@@
     (effects (font (size 1.27 1.27)) (justify left))
   )
-  (hierarchical_label "COL3" (shape input) (at 88.9 83.82 180)
-    (effects (font (size 1.27 1.27)) (justify right))
-  )
-  (hierarchical_label "ROW1" (shape input) (at 124.46 76.2 0)
-    (effects (font (size 1.27 1.27)) (justify left))
+  (hierarchical_label "COL3" (shape input) (at 88.9 76.2 180)
+    (effects (font (size 1.27 1.27)) (justify right))
+  )
+  (hierarchical_label "ROW1" (shape input) (at 88.9 81.28 180)
+    (effects (font (size 1.27 1.27)) (justify right))
   )
   (hierarchical_label "COL3" (shape input) (at 224.79 30.48 90)
@@
       (effects (font (size 0.508 0.508)))
     )
-    (property "Footprint" "" (id 2) (at 177.165 43.815 0)
+    (property "Footprint" "MX_Only:MXOnly-1U-NoLED" (id 2) (at 177.165 43.815 0)
       (effects (font (size 1.524 1.524)) hide)
     )
@@
       (effects (font (size 1.27 1.27)) (justify right))
     )
-    (property "Footprint" "" (id 2) (at 204.47 90.17 90)
+    (property "Footprint" "Diode_SMD:D_SOD-123" (id 2) (at 204.47 90.17 90)
       (effects (font (size 1.27 1.27)) hide)
     )
@@
       (effects (font (size 0.508 0.508)))
     )
-    (property "Footprint" "" (id 2) (at 191.135 62.865 0)
+    (property "Footprint" "MX_Only:MXOnly-1U-NoLED" (id 2) (at 191.135 62.865 0)
       (effects (font (size 1.524 1.524)) hide)
     )
@@
       (effects (font (size 1.27 1.27)) (justify right))
     )
-    (property "Footprint" "" (id 2) (at 176.53 52.07 90)
+    (property "Footprint" "Diode_SMD:D_SOD-123" (id 2) (at 176.53 52.07 90)
       (effects (font (size 1.27 1.27)) hide)
     )
@@
       (effects (font (size 1.524 1.524)))
     )
-    (property "Value" "" (id 1) (at 106.68 54.61 0)
-      (effects (font (size 1.524 1.524)))
-    )
-    (property "Footprint" "" (id 2) (at 133.35 135.89 90)
+    (property "Value" "ProMicro" (id 1) (at 106.68 54.61 0)
+      (effects (font (size 1.524 1.524)))
+    )
+    (property "Footprint" "Keebio-Parts:ArduinoProMicro" (id 2) (at 133.35 135.89 90)
       (effects (font (size 1.524 1.524)) hide)
     )
@@
       (effects (font (size 0.508 0.508)))
     )
-    (property "Footprint" "" (id 2) (at 163.195 43.815 0)
+    (property "Footprint" "MX_Only:MXOnly-1U-NoLED" (id 2) (at 163.195 43.815 0)
       (effects (font (size 1.524 1.524)) hide)
     )
@@
       (effects (font (size 0.508 0.508)))
     )
-    (property "Footprint" "" (id 2) (at 191.135 43.815 0)
+    (property "Footprint" "MX_Only:MXOnly-1U-NoLED" (id 2) (at 191.135 43.815 0)
       (effects (font (size 1.524 1.524)) hide)
     )
@@
       (effects (font (size 1.27 1.27)) (justify right))
     )
-    (property "Footprint" "" (id 2) (at 204.47 52.07 90)
+    (property "Footprint" "Diode_SMD:D_SOD-123" (id 2) (at 204.47 52.07 90)
       (effects (font (size 1.27 1.27)) hide)
     )
@@
       (effects (font (size 0.508 0.508)))
     )
-    (property "Footprint" "" (id 2) (at 177.165 62.865 0)
+    (property "Footprint" "MX_Only:MXOnly-1U-NoLED" (id 2) (at 177.165 62.865 0)
       (effects (font (size 1.524 1.524)) hide)
     )
@@
       (effects (font (size 1.27 1.27)) hide)
     )
-    (property "Value" "" (id 1) (at 128.27 60.96 0))
+    (property "Value" "+5V" (id 1) (at 128.27 60.96 0))
     (property "Footprint" "" (id 2) (at 128.27 66.04 0)
       (effects (font (size 1.27 1.27)) hide)
@@
       (effects (font (size 1.27 1.27)) (justify right))
     )
-    (property "Footprint" "" (id 2) (at 204.47 71.12 90)
+    (property "Footprint" "Diode_SMD:D_SOD-123" (id 2) (at 204.47 71.12 90)
       (effects (font (size 1.27 1.27)) hide)
     )
@@
       (effects (font (size 0.508 0.508)))
     )
-    (property "Footprint" "" (id 2) (at 163.195 62.865 0)
+    (property "Footprint" "MX_Only:MXOnly-1U-NoLED" (id 2) (at 163.195 62.865 0)
       (effects (font (size 1.524 1.524)) hide)
     )
@@
     (in_bom yes) (on_board yes) (fields_autoplaced)
     (property "Reference" "SW1" (id 0) (at 137.16 55.88 0))
-    (property "Value" "" (id 1) (at 137.16 58.42 0))
-    (property "Footprint" "" (id 2) (at 137.16 58.42 0)
+    (property "Value" "SW_Push" (id 1) (at 137.16 58.42 0))
+    (property "Footprint" "Keebio-Parts:SW_Tactile_SPST_Angled_MJTP1117-no-mount" (id 2) (at 137.16 58.42 0)
       (effects (font (size 1.27 1.27)) hide)
     )
@@
       (effects (font (size 1.27 1.27)) (justify right))
     )
-    (property "Footprint" "" (id 2) (at 190.5 52.07 90)
+    (property "Footprint" "Diode_SMD:D_SOD-123" (id 2) (at 190.5 52.07 90)
       (effects (font (size 1.27 1.27)) hide)
     )
@@
       (effects (font (size 0.508 0.508)))
     )
-    (property "Footprint" "" (id 2) (at 205.105 62.865 0)
+    (property "Footprint" "MX_Only:MXOnly-1U-NoLED" (id 2) (at 205.105 62.865 0)
       (effects (font (size 1.524 1.524)) hide)
     )
@@
       (effects (font (size 1.27 1.27)) hide)
     )
-    (property "Value" "" (id 1) (at 146.05 68.58 0))
+    (property "Value" "GND" (id 1) (at 146.05 68.58 0))
     (property "Footprint" "" (id 2) (at 146.05 63.5 0)
       (effects (font (size 1.27 1.27)) hide)
@@
       (effects (font (size 1.27 1.27)) (justify right))
     )
-    (property "Footprint" "" (id 2) (at 190.5 71.12 90)
+    (property "Footprint" "Diode_SMD:D_SOD-123" (id 2) (at 190.5 71.12 90)
       (effects (font (size 1.27 1.27)) hide)
     )
@@
       (effects (font (size 1.27 1.27)) (justify right))
     )
-    (property "Footprint" "" (id 2) (at 218.44 71.12 90)
+    (property "Footprint" "Diode_SMD:D_SOD-123" (id 2) (at 218.44 71.12 90)
       (effects (font (size 1.27 1.27)) hide)
     )
@@
       (effects (font (size 1.27 1.27)) (justify right))
     )
-    (property "Value" "" (id 1) (at 179.07 72.3899 90)
-      (effects (font (size 1.27 1.27)) (justify right))
-    )
-    (property "Footprint" "" (id 2) (at 176.53 71.12 90)
+    (property "Value" "D_Small" (id 1) (at 179.07 72.3899 90)
+      (effects (font (size 1.27 1.27)) (justify right))
+    )
+    (property "Footprint" "Diode_SMD:D_SOD-123" (id 2) (at 176.53 71.12 90)
       (effects (font (size 1.27 1.27)) hide)
     )
@@
       (effects (font (size 0.508 0.508)))
     )
-    (property "Footprint" "" (id 2) (at 216.535 81.915 0)
+    (property "Footprint" "MX_Only:MXOnly-1U-NoLED" (id 2) (at 216.535 81.915 0)
       (effects (font (size 1.524 1.524)) hide)
     )
@@
       (effects (font (size 1.27 1.27)) (justify right))
     )
-    (property "Footprint" "" (id 2) (at 229.87 90.17 90)
+    (property "Footprint" "Diode_SMD:D_SOD-123" (id 2) (at 229.87 90.17 90)
       (effects (font (size 1.27 1.27)) hide)
     )
@@
       (effects (font (size 1.27 1.27)) (justify right))
     )
-    (property "Footprint" "" (id 2) (at 218.44 90.17 90)
+    (property "Footprint" "Diode_SMD:D_SOD-123" (id 2) (at 218.44 90.17 90)
       (effects (font (size 1.27 1.27)) hide)
     )
@@
       (effects (font (size 0.508 0.508)))
     )
-    (property "Footprint" "" (id 2) (at 205.105 81.915 0)
-      (effects (font (size 1.524 1.524)) hide)
-    )
+    (property "Footprint" "MX_Only:MXOnly-1U-NoLED" (id 2) (at 205.105 81.915 0)
+      (effects (font (size 1.524 1.524)) hide)
+    )
